File: Hardware/gwxcontrol-mainboard/gwxcontrol-mainboard.kicad_pcb (KiCad board)
At the start: 2 copper layers, 29 parts, among them J1 8P8C, J10 Conn_02x08_Odd_Even, J11 Conn_02x08_Odd_Even, J12 Conn_02x08_Odd_Even, J13 Conn_02x08_Odd_Even, J2 8P8C, J3 8P8C, J4 8P8C, J5 Screw_Terminal_01x02, J6 Screw_Terminal_01x02, J7 Screw_Terminal_01x04, J8 Screw_Terminal_01x04, J9 8P8C, U1 ULN2803A, U2 PCF8574T, U3 ULN2803A, U4 YAAJ_WeAct_BlackPill_Part_Lik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

Commit message: Changed to 2x8 connector
Connections:
- J10 pad 1: unconnected-(J10-Pin_1-Pad1) -> GND
- J10 pad 7: /E1A.U -> /E1A.D
- J10 pad 9: /E1A.D -> /E1A.U
- J11 pad 7: /E1B.U -> /E1B.D
- J11 pad 9: /E1B.D -> /E1B.U
- J12 pad 7: /E2A.U -> /E2A.D
- J12 pad 9: /E2A.D -> /E2A.U
- J13 pad 7: /E2B.U -> /E2B.D
- J13 pad 9: /E2B.D -> /E2B.U

Commit message: Pins for water and wind
Parts:
- removed R1: R, Resistor_SMD:R_0603_1608Metric_Pad0.98x0.95mm_HandSolder
- added D2: BAT54CW, Package_TO_SOT_SMD:SOT-323_SC-70, F.Cu at (126.5, 55.7)
- added R4: 4k7, Resistor_SMD:R_0603_1608Metric_Pad0.98x0.95mm_HandSolder, F.Cu at (126.3, 58.7)
- added R5: 4k7, Resistor_SMD:R_0603_1608Metric_Pad0.98x0.95mm_HandSolder, F.Cu at (126.3, 61.2)
Connections:
- net /M1Up renamed /M1up
- net //M1Up renamed //M1up
- net Net-(U1-I1) renamed /M1A
- J3 pad 5: unconnected-(J3-Pad5) -> //D1
- J3 pad 6: unconnected-(J3-Pad6) -> //D2
- U3 pad 13: //D2 -> unconnected-(U3-O6-Pad13)
- U3 pad 14: //D1 -> unconnected-(U3-O5-Pad14)
- U3 pad 5: /D1 -> unconnected-(U3-I5-Pad5)
- U3 pad 6: /D2 -> unconnected-(U3-I6-Pad6)
- U4 pad 10: unconnected-(U4-PA15-Pad10) -> /E2A.U
- U4 pad 11: unconnected-(U4-PB3-Pad11) -> /E2A.D
- U4 pad 12: unconnected-(U4-PB4-Pad12) -> /E2B.U
- U4 pad 13: unconnected-(U4-PB5-Pad13) -> /E2B.D
- U4 pad 3: unconnected-(U4-PB14-Pad3) -> /wind
- U4 pad 34: unconnected-(U4-PB0-Pad34) -> /W1
- U4 pad 35: unconnected-(U4-PB1-Pad35) -> /W2
- U4 pad 36: unconnected-(U4-PB2-Pad36) -> /W3
- U4 pad 37: unconnected-(U4-PB10-Pad37) -> /W4
- U4 pad 4: unconnected-(U4-PB15-Pad4) -> /E1A.U
- U4 pad 5: unconnected-(U4-PA8-Pad5) -> /E1A.D
- U4 pad 8: unconnected-(U4-PA11-Pad8) -> /E1B.U
- U4 pad 9: unconnected-(U4-PA12-Pad9) -> /E1B.D
