File: Hardware/gwxcontrol-mainboard/gwxcontrol-mainboard.kicad_sch (KiCad schematic)
At the start: 29 parts, among them J1 8P8C, J10 Conn_02x08_Odd_Even, J11 Conn_02x08_Odd_Even, J12 Conn_02x08_Odd_Even, J13 Conn_02x08_Odd_Even, J2 8P8C, J3 8P8C, J4 8P8C, J5 Screw_Terminal_01x02, J6 Screw_Terminal_01x02, J7 Screw_Terminal_01x04, J8 Screw_Terminal_01x04, J9 8P8C, U1 ULN2803A, U2 PCF8574T, U3 ULN2803A, U4 YAAJ_WeAct_BlackPill_Part_Lik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

Commit message: Changed to 2x8 connector
Connections:
- net E1A.D: now also J10.7 (Pin_7); no longer J10.9 (Pin_9)
- net E1A.U: now also J10.9 (Pin_9); no longer J10.7 (Pin_7)
- net E1B.D: now also J11.7 (Pin_7); no longer J11.9 (Pin_9)
- net E1B.U: now also J11.9 (Pin_9); no longer J11.7 (Pin_7)
- net E2A.D: now also J12.7 (Pin_7); no longer J12.9 (Pin_9)
- net E2A.U: now also J12.9 (Pin_9); no longer J12.7 (Pin_7)
- net E2B.D: now also J13.7 (Pin_7); no longer J13.9 (Pin_9)
- net E2B.U: now also J13.9 (Pin_9); no longer J13.7 (Pin_7)
- net GND: now also J10.1 (Pin_1)
Changed lines of the file:
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@@
 	)
 	(junction
+		(at 172.72 59.69)
+		(diameter 0)
+		(color 0 0 0 0)
+	)
+	(junction
 		(at 177.8 78.74)
 		(diameter 0)
@@
 	(wire
 		(pts
+			(xy 172.72 59.69) (xy 199.39 59.69)
+		)
+		(stroke
+			(width 0)
+			(type default)
+		)
+	)
+	(wire
+		(pts
 			(xy 247.65 55.88) (xy 256.54 55.88)
 		)
@@
 	(wire
 		(pts
+			(xy 172.72 59.69) (xy 172.72 60.96)
+		)
+		(stroke
+			(width 0)
+			(type default)
+		)
+	)
+	(wire
+		(pts
 			(xy 157.48 57.15) (xy 177.8 57.15)
 		)
@@
 	(wire
 		(pts
-			(xy 167.64 59.69) (xy 199.39 59.69)
+			(xy 167.64 59.69) (xy 172.72 59.69)
 		)
 		(stroke
@@
 		)
 	)
+	(label "E2A.U"
+		(at 168.91 100.33 0)
+		(effects
+			(font
+				(size 1.27 1.27)
+			)
+			(justify left bottom)
+		)
+	)
 	(label "{slash}W2"
 		(at 240.03 135.89 0)
@@
 		)
 	)
-	(label "E2A.U"
-		(at 176.53 101.6 0)
-		(effects
-			(font
-				(size 1.27 1.27)
-			)
-			(justify left bottom)
-		)
-	)
 	(label "M2A"
 		(at 124.46 102.87 0)
@@
 		)
 	)
-	(label "E1B.U"
-		(at 170.18 77.47 0)
+	(label "M1+"
+		(at 250.19 38.1 0)
 		(effects
 			(font
@@
 		)
 	)
-	(label "M1+"
-		(at 250.19 38.1 0)
+	(label "E2A.D"
+		(at 175.26 101.6 0)
+		(effects
+			(font
+				(size 1.27 1.27)
+			)
+			(justify left bottom)
+		)
+	)
+	(label "E2B.D"
+		(at 170.18 125.73 0)
 		(effects
 			(font
@@
 		)
 	)
-	(label "M2A+"
-		(at 186.69 100.33 0)
+	(label "E2B.U"
+		(at 177.8 124.46 0)
 		(effects
 			(font
@@
 		)
 	)
-	(label "E1B.D"
-		(at 177.8 76.2 0)
+	(label "M2A+"
+		(at 186.69 100.33 0)
 		(effects
 			(font
@@
 		)
 	)
-	(label "E1A.D"
-		(at 176.53 52.07 0)
-		(effects
-			(font
-				(size 1.27 1.27)
-			)
-			(justify left bottom)
-		)
-	)
 	(label "{slash}M1Up"
 		(at 162.56 78.74 0)
@@
 		)
 	)
+	(label "E1B.U"
+		(at 177.8 76.2 0)
+		(effects
+			(font
+				(size 1.27 1.27)
+			)
+			(justify left bottom)
+		)
+	)
 	(label "SCL2"
 		(at 72.39 115.57 0)
@@
 		)
 	)
-	(label "E2A.D"
-		(at 170.18 100.33 0)
-		(effects
-			(font
-				(size 1.27 1.27)
-			)
-			(justify left bottom)
-		)
-	)
 	(label "W2"
 		(at 213.36 135.89 0)
@@
 		)
 	)
-	(label "SDA2"
-		(at 72.39 118.11 0)
+	(label "E1A.U"
+		(at 173.99 52.07 0)
 		(effects
 			(font
@@
 		)
 	)
-	(label "E1A.U"
-		(at 176.53 22.86 0)
+	(label "SDA2"
+		(at 72.39 118.11 0)
 		(effects
 			(font
@@
 		)
 	)
-	(label "{slash}M1B"
-		(at 149.86 100.33 0)
+	(label "E1A.U"
+		(at 176.53 22.86 0)
 		(effects
 			(font
@@
 		)
 	)
-	(label "E2B.U"
-		(at 176.53 38.1 0)
+	(label "{slash}M1B"
+		(at 149.86 100.33 0)
 		(effects
 			(font
@@
 	)
 	(label "E2B.U"
-		(at 168.91 125.73 0)
+		(at 176.53 38.1 0)
 		(effects
 			(font
@@
 		)
 	)
-	(label "E2B.D"
-		(at 175.26 124.46 0)
-		(effects
-			(font
-				(size 1.27 1.27)
-			)
-			(justify left bottom)
-		)
-	)
 	(label "SDA1"
 		(at 72.39 113.03 0)
@@
 		)
 	)
-	(label "E1A.U"
-		(at 168.91 53.34 0)
-		(effects
-			(font
-				(size 1.27 1.27)
-			)
-			(justify left bottom)
-		)
-	)
 	(label "SCL1"
 		(at 72.39 110.49 0)
@@
 	)
 	(label "E1B.D"
+		(at 170.18 77.47 0)
+		(effects
+			(font
+				(size 1.27 1.27)
+			)
+			(justify left bottom)
+		)
+	)
+	(label "E1B.D"
 		(at 176.53 30.48 0)
 		(effects
@@
 		(effects
 			(font
+				(size 1.27 1.27)
+			)
+			(justify left bottom)
+		)
+	)
+	(label "E1A.D"
+		(at 167.64 53.34 0)
+		(effects
+			(font

Commit message: Pins for water and wind
Parts:
- removed R1: R, Resistor_SMD:R_0603_1608Metric_Pad0.98x0.95mm_HandSolder, symbol Device:R
- added D2: BAT54CW, Package_TO_SOT_SMD:SOT-323_SC-70, symbol Diode:BAT54CW
- added R4, R5: 4k7, Resistor_SMD:R_0603_1608Metric_Pad0.98x0.95mm_HandSolder, symbol Device:R
Connections:
- net +5V: now also D2.3, R4.2, R5.1
- net D1: no longer U3.5 (I5)
- net D2: no longer U3.6 (I6)
- net E1A.D: now also U4.5 (PA8)
- net E1A.U: now also U4.4 (PB15)
- net E1B.D: now also U4.9 (PA12)
- net E1B.U: now also U4.8 (PA11)
- net E2A.D: now also U4.11 (PB3)
- net E2A.U: now also U4.10 (PA15)
- net E2B.D: now also U4.13 (PB5)
- net E2B.U: now also U4.12 (PB4)
- net M1A: now also U1.1 (I1), U4.33 (PA7)
- net W1: now also U4.34 (PB0)
- net W2: now also U4.35 (PB1)
- net W3: now also U4.36 (PB2)
- net W4: now also U4.37 (PB10)
- net wind: now also U4.3 (PB14)
- net /D1: now also J3.5; no longer U3.14 (O5)
- net /D2: now also J3.6; no longer U3.13 (O6)
- net /M2up: now also D2.2, R5.2
- net M1Up renamed M1up
- net /M1Up renamed /M1up
- net /M1up: now also D2.1, R4.1
Other:
- note added: "Motors Direction Relais"
- note added: "PC14/15: RCT-XTAL"
- note added: "Thermo/Hygro-Sensors"
- note removed: "Motors Direction"
- moved on the sheet: A1, J3, U4

Commit message: pins changed
Connections:
- net W1: now also U4.2 (PB13); no longer U4.34 (PB0)
- net W2: now also U4.1 (PB12); no longer U4.35 (PB1)
Changed lines of the file:
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@@
-	(wire
-		(pts
-			(xy 114.3 90.17) (xy 116.84 90.17)
-		)
-		(stroke
-			(width 0)
-			(type default)
-		)
-	)
 	(wire
 		(pts
@@
 	(wire
 		(pts
+			(xy 68.58 80.01) (xy 64.77 80.01)
+		)
+		(stroke
+			(width 0)
+			(type default)
+		)
+	)
+	(wire
+		(pts
 			(xy 106.68 180.34) (xy 106.68 182.88)
 		)
@@
 	(wire
 		(pts
-			(xy 114.3 92.71) (xy 118.11 92.71)
+			(xy 68.58 77.47) (xy 66.04 77.47)
 		)
 		(stroke
@@
 		)
 	)
+	(label "W1"
+		(at 67.31 80.01 180)
+		(effects
+			(font
+				(size 1.27 1.27)
+			)
+			(justify right bottom)
+		)
+	)
 	(label "SCL1"
 		(at 63.5 35.56 90)
@@
 		)
 	)
-	(label "W1"
-		(at 115.57 92.71 0)
-		(effects
-			(font
-				(size 1.27 1.27)
-			)
-			(justify left bottom)
-		)
-	)
 	(label "{slash}M1up"
 		(at 171.45 57.15 0)
@@
 		)
 	)
-	(label "W2"
-		(at 115.57 90.17 0)
-		(effects
-			(font
-				(size 1.27 1.27)
-			)
-			(justify left bottom)
-		)
-	)
 	(label "{slash}M1up"
 		(at 162.56 78.74 0)
@@
 		)
 	)
+	(label "W2"
+		(at 67.31 77.47 180)
+		(effects
+			(font
+				(size 1.27 1.27)
+			)
+			(justify right bottom)
+		)
+	)
