File: Hardware/3-Phase-Motorcontroller/simple/gwx-control.kicad_sch (KiCad schematic)
At the start: 38 parts, among them IC1 74LS02D, IC2 74123D, J1 MTA07-100, T1 BC850, T2 BC850

Commit message: Changed to 2x8 connector
Parts:
- removed IC1: 74LS02D, gwx-control:SO14, symbol gwx-control-eagle-import:7402D
- removed IC2: 74123D, gwx-control:SO16, symbol gwx-control-eagle-import:74123D
- removed J1: MTA07-100, gwx-control:10X07MTA, symbol gwx-control-eagle-import:MTA07-100
- added J10: Conn_02x08_Odd_Even, Connector_PinHeader_2.54mm:PinHeader_2x08_P2.54mm_Horizontal, symbol Connector_Generic:Conn_02x08_Odd_Even
- added U1: 74LS02, Package_SO:SOIC-14_3.9x8.7mm_P1.27mm, symbol 74xx:74LS02
- added U2: 74LS123, Package_SO:SOIC-16_3.9x9.9mm_P1.27mm, symbol 74xx:74LS123
Connections:
- net /END_DOWN: now also U1.6
- net /END_UP: now also U1.11
- net /MOTOR_OK: now also U2.5 (Q)
- net /MOTOR_ON: now also J10.3 (Pin_3)
- net /OK: now also J10.13 (Pin_13), U1.1
- net /Q: now also U2.12 (~{Q})
- net /UP: now also J10.5 (Pin_5), U1.12, U1.8, U1.9
- net GND: now also J10.1 (Pin_1), J10.16 (Pin_16), J10.2 (Pin_2), U1.7 (GND), U2.1 (A), U2.2 (B), U2.8 (GND), U2.9 (A)
- net MOTOR_ON+: now also J10.11 (Pin_11)
- net VCC: now also J10.15 (Pin_15), U2.11 (Clr), U2.16 (VCC)
- net at R16.2: now also J10.7 (Pin_7)
- net at R15.2: now also J10.9 (Pin_9)
- net at D3.3 (CC), R9.1: now also U2.10 (B)
- net at C4.+, R6.2: now also U2.15 (RCext)
- net at C3.+, R5.1: now also U2.7 (RCext)
- net at C3.-: now also U2.6 (Cext)
- net at C4.-: now also U2.14 (Cext)
- new net: U1.13, U1.2
- new net: U1.3, U1.4
- new net: U1.10, U1.5
Other:
- moved on the sheet: C1, C2, C7

Commit message: LEDs libs updated
Parts:
- removed LED1, LED2, LED3, LED4, LED5: LED_ESML0603, LED_SMD:LED_0603_1608Metric_Pad1.05x0.95mm_HandSolder, symbol gwx-control-eagle-import:LED_ESML0603
- added C8: 47µ, Capacitor_THT:CP_Radial_D8.0mm_P5.00mm, symbol gwx-control-eagle-import:CPOL-EUE5-6
- added D4, D5, D6, D7, D8: LED_ESML0603, LED_SMD:LED_0603_1608Metric_Pad1.05x0.95mm_HandSolder, symbol Device:LED
- C1, C2, C5, C6, C7: footprint gwx-control:C0603K -> Capacitor_SMD:C_0603_1608Metric
- C3: footprint gwx-control:E5-6 -> Capacitor_Tantalum_SMD:CP_EIA-6032-28_Kemet-C_HandSolder
- C4: value CPOL-EUE5-6 -> 47µ; footprint gwx-control:E5-6 -> Capacitor_Tantalum_SMD:CP_EIA-6032-28_Kemet-C_HandSolder
- D2, D3: footprint gwx-control:SOT23 -> Package_TO_SOT_SMD:TSOT-23
- R1, R10, R3, R4, R5, R6, R7, R8, R9: footprint gwx-control:R0603 -> Resistor_SMD:R_0603_1608Metric_Pad0.98x0.95mm_HandSolder
- T1, T2: footprint gwx-control:SOT23-BEC -> Package_TO_SOT_SMD:TSOT-23
Connections:
- net /END_DOWN: now also D8.1 (K)
- net /END_UP: now also D7.1 (K)
- net /MOTOR_OK: now also D5.1 (K)
- net /MOTOR_ON: now also D4.1 (K)
- net /UP: now also D6.1 (K)
- net at R1.1: now also D8.2 (A)
- net at C3.-, U2.6 (Cext): now also C8.-
- net at C3.+, R5.1, U2.7 (RCext): now also C8.+
- net at R14.1: now also D6.2 (A)
- net at R12.1: now also D5.2 (A)
- net at R11.1: now also D4.2 (A)
- net at R2.1: now also D7.2 (A)

Commit message: PCB shrinked
Parts:
- removed D1: 1N4148, gwx-control:DO35-10, symbol gwx-control-eagle-import:1N4148DO35-10
- removed R18: 4k7, Resistor_SMD:R_0603_1608Metric_Pad0.98x0.95mm_HandSolder, symbol gwx-control-eagle-import:resistor_R-EU_R0603
- added C10, C9: 100n, Capacitor_SMD:C_0603_1608Metric, symbol gwx-control-eagle-import:C-EUC0603K
Connections:
- net /END_DOWN: now also C10.1
- net /END_UP: now also C9.2
- net GND: now also C10.2, C9.1
